Commit message: minimal working moveit

File: igus_axis_description/urdf/igus_axis_macro.xacro (robot description, xacro)
@@ -77,5 +77,5 @@
     <parent link="${prefix}link1"/>
     <child link="${prefix}${axisend_link}"/>
-    <origin xyz="0 ${width1y/2} ${height2/2}" rpy="0 0 0"/>
+    <origin xyz="0 0 0" rpy="0 0 0"/>
     <axis xyz="0 0 1"/>
     <dynamics damping="0.7"/>

File: igus_axis_description/urdf/igus_axis_standalone.urdf.xacro (robot description, xacro)
@@ -7,8 +7,9 @@
 <robot xmlns:xacro="http://www.ros.org/wiki/xacro" name="2dof_robot">
   <!-- Used for fixing robot -->
-<link name="base_link"/>
-<xacro:arg name="axisparent" default="base_link" />
-<xacro:arg name="prefix" default="axis_" />
-<xacro:arg name="axisend_link" default="end_link" />
-  <xacro:include filename="$(find igus_axis_description)/urdf/igus_axis_description.urdf.xacro" />
+<link name="world"/>
+  <joint name="joint_world_to_base" type="fixed">
+    <parent link="world"/>
+    <child link="base_link" />
+  </joint>
+  <xacro:include filename="$(find igus_axis_description)/urdf/igus_axis.urdf.xacro" />
 </robot>
