Commit message: launch file, add multiple yaml files etc

File: igus_axis_description/urdf/igus_axis.ros2_control.xacro (robot description, xacro)
@@ -16,9 +16,10 @@
       </hardware>
       <joint name="${prefix}joint1">
-        <command_interface name="position">
+        <command_interface name="velocity">
           <param name="min">0</param>
           <param name="max">2</param>
         </command_interface>
         <state_interface name="position"/>
+        <state_interface name="velocity"/>
       </joint>
       <!-- <joint name="${prefix}joint2">

File: igus_axis_description/urdf/igus_axis_macro.xacro (robot description, xacro)
@@ -48,5 +48,5 @@
     <axis xyz="0 0 1"/>
     <dynamics damping="0.7"/>
-    <limit lower="0" upper="2" velocity="100" effort="100"/>
+    <limit lower="0" upper="2" velocity=".1" effort="100"/>
   </joint>
   <!-- Middle Link -->

File: martha_driver/urdf/martha.urdf.xacro (robot description, xacro)
@@ -6,9 +6,16 @@
 <xacro:arg name="axisend_link" default="end_link" />
 <xacro:arg name="prefix" default="axis_" />
+<joint name="connector" type="fixed">
+    <parent link="$(arg prefix)end_link" />
+    <child link="basething" />
+    <origin xyz="0 0 0" rpy="${-0.5*pi} ${0.25*pi} 0"/>
+</joint>
+<link name="basething">
+    </link>
 <!-- <link name="base_link"/> -->
-<xacro:arg name="parent" default="axis_end_link" />
+<xacro:arg name="parent" default="basething" />
 <xacro:arg name="tf_prefix" default="UR_" />
 <xacro:arg name="name" default="x" />
 <xacro:include filename="$(find igus_axis_description)/urdf/igus_axis_description.urdf.xacro" />
-<xacro:include filename="$(find ur10e_description)/urdf/ur_description.urdf.xacro" />
+<!-- <xacro:include filename="$(find ur10e_description)/urdf/ur_description.urdf.xacro" /> -->
 </robot>

File: ur10e_description/urdf/ur.urdf.xacro (robot description, xacro)
@@ -1,5 +1,10 @@
 <?xml version="1.0"?>
 <robot xmlns:xacro="http://www.ros.org/wiki/xacro" name="2dof_robot">
-<!-- <link name="world" /> -->
+<link name="world" />
+<joint name="world_to_base_joint" type="fixed">
+    <parent link="world" />
+    <child link="base_link" />
+    <origin xyz="0 0 0" rpy="0 0 0"/>
+</joint>
 <link name="base_link"/>
 <xacro:arg name="parent" default="base_link" />

Commit message: minimum working jtc

File: igus_axis_description/urdf/igus_axis.ros2_control.xacro (robot description, xacro)
@@ -23,11 +23,4 @@
         <state_interface name="velocity"/>
       </joint>
-      <!-- <joint name="${prefix}joint2">
-        <command_interface name="position">
-          <param name="min">-1</param>
-          <param name="max">1</param>
-        </command_interface>
-        <state_interface name="position"/>
-      </joint> -->
     </ros2_control>
   </xacro:macro>

File: igus_axis_description/urdf/igus_axis_macro.xacro (robot description, xacro)
@@ -48,5 +48,5 @@
     <axis xyz="0 0 1"/>
     <dynamics damping="0.7"/>
-    <limit lower="0" upper="2" velocity=".1" effort="100"/>
+    <limit lower="0" upper="2" velocity=".05" effort="10"/>
   </joint>
   <!-- Middle Link -->

File: martha_driver/urdf/martha.urdf.xacro (robot description, xacro)
@@ -18,4 +18,4 @@
 <xacro:arg name="name" default="x" />
 <xacro:include filename="$(find igus_axis_description)/urdf/igus_axis_description.urdf.xacro" />
-<!-- <xacro:include filename="$(find ur10e_description)/urdf/ur_description.urdf.xacro" /> -->
+<xacro:include filename="$(find ur10e_description)/urdf/ur_description.urdf.xacro" />
 </robot>

File: ur10e_description/urdf/ur_conform.urdf.xacro (robot description, xacro)
@@ -1,6 +1,11 @@
 <?xml version="1.0"?>
 <robot xmlns:xacro="http://www.ros.org/wiki/xacro" name="2dof_robot">
-<link name="world" />
-<xacro:arg name="parent" default="world" />
+<!-- <link name="world" />  -->
+<!-- <joint name="first_k" type="fixed">
+    <parent link="world">
+    <child link="base_link">
+</joint> -->
+<link name="base_link" />
+<xacro:arg name="parent" default="base_link" />
 <xacro:arg name="tf_prefix" default="" />
 <xacro:include filename="$(find ur10e_description)/urdf/ur_description.urdf.xacro" />

Commit message: working moveit

File: igus_axis_description/urdf/igus_axis.ros2_control.xacro (robot description, xacro)
@@ -1,6 +1,6 @@
 <?xml version="1.0"?>
 <robot xmlns:xacro="http://www.ros.org/wiki/xacro">
-  <xacro:macro name="rrbot_ros2_control" params="name prefix">
-    <ros2_control name="${name}" type="system">
+  <xacro:macro name="rrbot_ros2_control" params="namae prefix axis_ip">
+    <ros2_control name="${namae}" type="system">
       <hardware>
         <plugin>igus_axis_driver/RRBotSystemPositionOnlyHardware</plugin>
@@ -8,5 +8,5 @@
         <param name="example_param_hw_stop_duration_sec">3.0</param>
         <param name="example_param_hw_slowdown">100</param>
-        <param name="ip">192.168.0.10</param>
+        <param name="ip">${axis_ip}</param>
         <param name="axisName">${prefix}joint1</param>
         <param name="port">502</param>

File: igus_axis_description/urdf/igus_axis.urdf.xacro (robot description, xacro)
@@ -11,4 +11,5 @@
 <xacro:arg name="prefix" default="axis_" />
 <xacro:arg name="axisend_link" default="end_link" />
+<xacro:arg name="axis_ip" default="192.168.0.10" />
   <xacro:include filename="$(find igus_axis_description)/urdf/igus_axis_description.urdf.xacro" />
 </robot>

File: igus_axis_description/urdf/igus_axis_description.urdf.xacro (robot description, xacro)
@@ -9,5 +9,4 @@
     <origin xyz="0 0 0" rpy="0 0 0" />
   </xacro:rrbot>
-  <xacro:rrbot_ros2_control
-    name="RRBot" prefix="$(arg prefix)" />
+  <xacro:rrbot_ros2_control    namae="RRBot" prefix="$(arg prefix)" axis_ip="$(arg axis_ip)" />
 </robot>

File: igus_axis_description/urdf/igus_axis_standalone.urdf.xacro (robot description, xacro)
@@ -5,5 +5,5 @@
 https://github.com/ros-simulation/gazebo_ros_demos/blob/kinetic-devel/rrbot_description/urdf/rrbot.xacro
 -->
-<robot xmlns:xacro="http://www.ros.org/wiki/xacro" name="2dof_robot">
+<robot xmlns:xacro="http://www.ros.org/wiki/xacro" name="igus_axis">
   <!-- Used for fixing robot -->
 <link name="world"/>

File: martha_driver/urdf/marthaEDIT.urdf.xacro (robot description, xacro)
@@ -18,5 +18,5 @@
 <link name="basething">
     </link>
-<xacro:arg name="parent" default="basething" />
+<xacro:arg name="parent" default="base_link" />
 <xacro:arg name="tf_prefix" default="UR_" />
 <xacro:include filename="$(find igus_axis_description)/urdf/igus_axis_description.urdf.xacro" />

File: ur10e_description/urdf/ur_description.urdf.xacro (robot description, xacro)
@@ -5,4 +5,6 @@
    <!-- import main macro -->
    <xacro:include filename="$(find ur10e_description)/urdf/ur_macro.xacro"/>
+   <xacro:include filename="$(find ur10e_description)/urdf/inc/ur_transmissions.xacro" />
+   <xacro:include filename="$(find ur10e_description)/urdf/inc/ur_common.xacro" />
    <!-- parameters -->
    <xacro:arg name="joint_limit_params" default="$(find ur10e_description)/config/joint_limits.yaml"/>

File: ur10e_description/urdf/ur_macro.xacro (robot description, xacro)
@@ -42,6 +42,4 @@
      - Muhammad Asif Rana
   -->
-  <xacro:include filename="$(find ur10e_description)/urdf/inc/ur_transmissions.xacro" />
-  <xacro:include filename="$(find ur10e_description)/urdf/inc/ur_common.xacro" />
   <xacro:macro name="ur_robot" params="
     name
